File: PCB/RH017.1/RH017.1.brd (EAGLE design)
At the start: 99.1 x 78.7 mm, 62 parts, among them CN1 USB, IC1 MPR121, U1 ATMega-328, U11 REG1117, X1 16 MHz

Commit message: updates
Connections:
- removed net VCC: R2.1
- new net GP9: MDL1.19
- new net GP_CSO: MDL1.17
- new net GP_MISO: MDL1.18
- new net GP_MOSI: MDL1.21
- new net GP_SCLK: MDL1.22
- net 3.3V: now also R2.1
- net GP10: now also MDL1.20
Routing:
- net GP10: track 0.00 -> 20.9 mm, vias 0 -> 2
- net KEY0: track 52.0 -> 50.0 mm
- net 3.3V: track 195.7 -> 197.4 mm
Changed lines of the file:
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@@
 <text x="6.5" y="52" size="0.8128" layer="25">GP15</text>
 <text x="6.5" y="51" size="0.8128" layer="25">GND</text>
+<circle x="23.8" y="20.3" radius="0.1" width="0.4064" layer="25"/>
+<circle x="62.1" y="41.6" radius="0.1" width="0.4064" layer="25"/>
 </plain>
 <attributes>
@@
 </element>
 <element name="U1" library="LowPowerLab" package="TQFP32-08" value="ATMega-328" x="28" y="16" smashed="yes">
-<attribute name="NAME" x="22.825" y="20.08" size="0.8128" layer="25"/>
+<attribute name="NAME" x="21.425" y="18.18" size="0.8128" layer="25"/>
 </element>
 <element name="C8" library="LowPowerLab" package="0603-CAP" value="0.1" x="25" y="8" smashed="yes">
@@
 <via x="19.0881" y="45.3771" extent="1-16" drill="0.3048"/>
 <via x="15.0876" y="28.2321" extent="1-16" drill="0.3048"/>
+<contactref element="R2" pad="1"/>
+<wire x1="9.375" y1="23.125" x2="10" y2="23.125" width="0.3048" layer="1"/>
+<wire x1="9.25" y1="23.25" x2="9.375" y2="23.125" width="0.3048" layer="1"/>
+<wire x1="9.25" y1="24" x2="9.25" y2="23.25" width="0.3048" layer="1"/>
+<wire x1="10" y1="23.125" x2="10" y2="23.1" width="0.3048" layer="1"/>
+<wire x1="9.25" y1="24" x2="9.2583" y2="24.1173" width="0.3048" layer="1"/>
 </signal>
 <signal name="VREG">
@@
 <contactref element="IC1" pad="8"/>
 <via x="83" y="63" extent="1-16" drill="0.306"/>
-<wire x1="83" y1="63" x2="76.5" y2="63" width="0.3048" layer="1"/>
-<wire x1="76.5" y1="63" x2="76.5" y2="57.5" width="0.3048" layer="1"/>
-<wire x1="76.5" y1="57.5" x2="77.5" y2="57.5" width="0.3048" layer="1"/>
-<wire x1="77.5" y1="57.5" x2="77.5" y2="54.5" width="0.3048" layer="1"/>
+<wire x1="83" y1="63" x2="77.5" y2="63" width="0.3048" layer="1"/>
+<wire x1="77.5" y1="63" x2="77.5" y2="54.5" width="0.3048" layer="1"/>
 <wire x1="77.5" y1="54.5" x2="76.5" y2="54.5" width="0.3048" layer="1"/>
 <wire x1="76.5" y1="54.5" x2="76.5" y2="35" width="0.3048" layer="1"/>
@@
 <via x="24.9174" y="26.9748" extent="1-16" drill="0.3048"/>
 </signal>
-<signal name="VCC">
-<contactref element="R2" pad="1"/>
-</signal>
 <signal name="GP10">
 <contactref element="SJ5" pad="1"/>
+<contactref element="MDL1" pad="20"/>
+<wire x1="22.25" y1="37.625" x2="22.25" y2="37" width="0.3048" layer="1"/>
+<wire x1="21.125" y1="37.625" x2="22.25" y2="37.625" width="0.3048" layer="1"/>
+<wire x1="20.875" y1="37.875" x2="21.125" y2="37.625" width="0.3048" layer="1"/>
+<wire x1="20.875" y1="39.375" x2="20.875" y2="37.875" width="0.3048" layer="1"/>
+<wire x1="21" y1="39.375" x2="20.875" y2="39.375" width="0.3048" layer="1"/>
+<wire x1="21.125" y1="39.375" x2="21" y2="39.375" width="0.3048" layer="16"/>
+<wire x1="24.875" y1="43.125" x2="21.125" y2="39.375" width="0.3048" layer="16"/>
+<wire x1="24.875" y1="45.875" x2="24.875" y2="43.125" width="0.3048" layer="16"/>
+<wire x1="31.5" y1="45.875" x2="24.875" y2="45.875" width="0.3048" layer="1"/>
+<wire x1="32" y1="46.375" x2="31.5" y2="45.875" width="0.3048" layer="1"/>
+<wire x1="32" y1="48" x2="32" y2="46.375" width="0.3048" layer="1"/>
+<wire x1="22.25" y1="37" x2="22.238" y2="37" width="0.3048" layer="1"/>
+<via x="21" y="39.375" extent="1-16" drill="0.3048"/>
+<via x="24.875" y="45.875" extent="1-16" drill="0.3048"/>
+</signal>
+<signal name="GP_CSO">
+<contactref element="MDL1" pad="17"/>
+</signal>
+<signal name="GP_MOSI">
+<contactref element="MDL1" pad="21"/>
+</signal>
+<signal name="GP_MISO">
+<contactref element="MDL1" pad="18"/>
+</signal>
+<signal name="GP_SCLK">
+<contactref element="MDL1" pad="22"/>
+</signal>
+<signal name="GP9">
+<contactref element="MDL1" pad="19"/>
 </signal>
 </signals>
